Commit message: Local file paths till retriever fixed

File: data/objects/plastic_bowl.urdf (robot description, URDF)
Before this commit: robot plastic_bowl, 1 links, 0 joints
Links:
- link /body: geometry collision mesh filename=plastic_bowl_collision.stl; visual mesh filename=plastic_bowl_visual.dae

File: data/objects/plastic_glass.urdf (robot description, URDF)
Before this commit: robot plastic_glass, 1 links, 0 joints
Links:
- link /body: geometry collision mesh filename=plastic_glass_collision.stl; visual mesh filename=plastic_glass_visual.dae

Commit message: Intermediate edits for aikido

File: data/objects/plastic_bowl.urdf (robot description, URDF)
Before this commit: robot plastic_bowl, 1 links, 0 joints
Links:
- link /body: geometry collision mesh filename=package://pr_ordata/data/objects/plastic_bowl_collision.stl; visual mesh filename=package://pr_ordata/data/objects/plastic_bowl_visual.dae

File: data/objects/plastic_glass.urdf (robot description, URDF)
Before this commit: robot plastic_glass, 1 links, 0 joints
Links:
- link /body: geometry collision mesh filename=package://pr_ordata/data/objects/plastic_glass_collision.stl; visual mesh filename=package://pr_ordata/data/objects/plastic_glass_visual.dae
