Commit message: add script converting kinbody into urdf

File: data/objects/block_bin.urdf (robot description, URDF)
Before this commit: robot block_bin, 1 links, 0 joints
Links:
- link base_link: geometry collision box size=0.01 0.3 0.15; collision box size=0.01 0.3 0.15

File: data/objects/box.urdf (robot description, URDF)
Before this commit: robot blue_wood_block_1inx1in, 1 links, 0 joints
Links:
- link base_link: geometry collision box size=0.2 0.29 0.11; visual box size=0.2 0.29 0.11
