Commit message: update converter and URDFs

File: data/objects/bin.urdf (robot description, URDF)
Before this commit: robot bin, 1 links, 0 joints
Links:
- removed link base_link
- added link bin_body; collision box size=0.01 0.58 0.17; collision box size=0.01 0.58 0.17

File: data/objects/block.urdf (robot description, URDF)
Before this commit: robot blue_wood_block_1inx1in, 1 links, 0 joints
Links:
- removed link base_link
- added link blue_wood_block_1inx1in; collision box size=0.0254 0.0254 0.0254; visual box size=0.0254 0.0254 0.0254

File: data/objects/block_bin.urdf (robot description, URDF)
Before this commit: robot block_bin, 1 links, 0 joints
Links:
- removed link base_link
- added link block_bin_body; collision box size=0.01 0.3 0.15; collision box size=0.01 0.3 0.15

File: data/objects/fuze_bottle.urdf (robot description, URDF)
Before this commit: robot fuze_bottle, 1 links, 0 joints
Links:
- removed link base_link
- added link fuze_bottle; collision mesh filename=fuze_bottle_collision.stl scale=0.10 0.10 0.10; visual mesh filename=fuze_bottle_visual.dae

File: data/objects/large_white_box.urdf (robot description, URDF)
Before this commit: robot large_white_box, 1 links, 0 joints
Links:
- removed link base_link
- added link large_white_box; collision box size=0.102 0.102 0.215; visual box size=0.102 0.102 0.215

File: data/objects/plastic_bowl.urdf (robot description, URDF)
Before this commit: robot plastic_bowl, 1 links, 0 joints
Links:
- removed link base_link
- added link plastic_bowl; collision mesh filename=plastic_bowl_collision.stl; visual mesh filename=plastic_bowl_visual.dae

File: data/objects/plate.urdf (robot description, URDF)
Before this commit: robot bowl, 1 links, 0 joints
Links:
- removed link bowl
- added link plate; collision mesh filename=plate.stl; visual mesh filename=plate.stl

File: data/objects/pop_tarts.urdf (robot description, URDF)
Before this commit: robot pop_tarts, 1 links, 0 joints
Links:
- removed link base_link
- added link pop_tarts; collision box size=0.1 0.1 0.14; collision sphere radius=0.1

File: data/objects/rubbermaid_ice_guard_pitcher.urdf (robot description, URDF)
Before this commit: robot rubbermaid_ice_guard_pitcher_blue, 1 links, 0 joints
Links:
- removed link base_link
- added link rubbermaid_ice_guard_pitcher_blue; collision mesh filename=rubbermaid_ice_guard_pitcher_mesh.stl; visual mesh filename=rubbermaid_ice_guard_pitcher_mesh.stl

File: data/objects/stamp.urdf (robot description, URDF)
Before this commit: robot paper_box, 1 links, 0 joints
Links:
- removed link paper_box
- added link stamp; collision cylinder length=0.20 radius=0.02; visual cylinder length=0.20 radius=0.02

File: data/objects/table.urdf (robot description, URDF)
Before this commit: robot table, 1 links, 0 joints
Links:
- removed link base_link
- added link table; collision box size=0.06 0.005 0.66; collision box size=0.06 0.005 0.66

File: data/objects/wicker_tray.urdf (robot description, URDF)
Before this commit: robot wicker_tray, 1 links, 0 joints
Links:
- removed link base_link
- added link wicker_tray; collision box size=0.02 0.65 0.12; collision box size=0.02 0.65 0.12

File: data/objects/wooden_table.urdf (robot description, URDF)
Before this commit: robot wooden_table, 1 links, 0 joints
Links:
- removed link base_link
- added link wooden_table; collision box size=0.7112 0.0508 0.69215; collision box size=0.7112 0.0508 0.69215
