Commit message: On branch tapo_demo_urdfs 	new file:   can.bak.urdf 	modified:   can.urdf 	new file:   can_collision.stl 	new file:   can_visual.dae 	new file:   model/__Metal_Aluminum_Anodized_.jpg 	new file:   model/__Metal_Aluminum_Anodized__0.jpg 	new file:   model/coladosentextur.jpg 	new file:   model/coladosentextur_1.jpg

File: data/objects/can.urdf (robot description, URDF)
Before this commit: robot can, 1 links, 0 joints
Links:
- link base_link: geometry collision mesh filename=can_collision.stl; visual mesh filename=can_visual.dae

Commit message: modified the urdf file to replace the stl  collision model with a cylinder primitive shape  Changes to be committed: 	modified:   can.urdf

File: data/objects/can.urdf (robot description, URDF)
Before this commit: robot can, 1 links, 0 joints
Links:
- link base_link: geometry collision cylinder length=0.123 radius=0.033; visual mesh filename=can_visual.dae
