Commit message: change origin of food_item and can

File: data/objects/food_item.urdf (robot description, URDF)
Before this commit: robot food_item, 1 links, 0 joints
Links:
- link food_item: geometry collision box size=0.025 0.025 0.015; visual box size=0.025 0.025 0.015

Commit message: disabled collision for food item (so it can be skewered

File: data/objects/food_item.urdf (robot description, URDF)
Before this commit: robot food_item, 1 links, 0 joints
Links:
- link food_item: geometry visual box size=0.025 0.025 0.015
