Commit message: pitcher things etc.

File: data/objects/rubbermaid_ice_guard_pitcher.urdf (robot description, URDF)
Before this commit: robot rubbermaid_ice_guard_pitcher_blue, 1 links, 0 joints
Links:
- link rubbermaid_ice_guard_pitcher_blue: geometry collision mesh filename=rubbermaid_ice_guard_pitcher_mesh.stl; visual mesh filename=new_pitcher.stl
