Commit message: modify sizes

File: data/objects/box.urdf (robot description, URDF)
Before this commit: robot paper_box, 1 links, 0 joints
Links:
- link paper_box: geometry collision box size=0.4 0.4 0.4; visual box size=0.4 0.4 0.4

File: data/objects/can.urdf (robot description, URDF)
Before this commit: robot can, 1 links, 0 joints
Links:
- link base_link: geometry collision cylinder length=0.8 radius=0.03; visual cylinder length=0.8 radius=0.03

Commit message: some more objects

File: data/objects/box.urdf (robot description, URDF)
Before this commit: robot paper_box, 1 links, 0 joints
Links:
- link paper_box: geometry collision box size=0.14 0.09 0.12; visual box size=0.14 0.09 0.12
