Commit message: updated tom's size

File: data/objects/tom.urdf (robot description, URDF)
Before this commit: robot tom, 1 links, 0 joints
Links:
- link base_link: geometry collision mesh filename=tom.dae scale=1 1 1; visual mesh filename=tom.dae scale=1 1 1

Commit message: wheelchair collision

File: data/objects/tom.urdf (robot description, URDF)
Before this commit: robot tom, 1 links, 0 joints
Links:
- link base_link: geometry collision mesh filename=tom.dae scale=1 1 1

Commit message: updated wheelchair and tom

File: data/objects/tom.urdf (robot description, URDF)
Before this commit: robot tom, 1 links, 0 joints
Links:
- link base_link: geometry collision box size=1.3 1.745 3; collision mesh filename=tom.dae scale=0.8 0.8 0.8

Commit message: Remove extra collision from Tom

File: data/objects/tom.urdf (robot description, URDF)
Before this commit: robot tom, 1 links, 0 joints
Links:
- link base_link: geometry collision mesh filename=tom.dae scale=0.8 0.8 0.8; visual mesh filename=tom.dae scale=0.8 0.8 0.8
