Commit message: Adding wheels to bookcase.urdf

File: data/furniture/bookcase.urdf (robot description, URDF)
Before this commit: robot bookcase, 1 links, 0 joints
Links:
- removed link base_link
- added link base_footprint, mass 0.1
- added link bookcase; collision mesh filename=bookcase.stl; visual mesh filename=bookcase.stl
- added link l_wheel_link; collision box size=0.02 0.03 0.0025; collision box size=0.02 0.03 0.0025
- added link r_wheel_link; collision box size=0.02 0.03 0.0025; collision box size=0.02 0.03 0.0025
Joints:
- added joint base_to_bookcase: type fixed, parent base_footprint, child bookcase, origin xyz=0.0 0.0 0.1125
- added joint base_to_l_wheel: type fixed, parent base_footprint, child l_wheel_link, origin xyz=0.738 0.2 0.1125 rpy=1.57 0 0
- added joint base_to_r_wheel: type fixed, parent base_footprint, child r_wheel_link, origin xyz=0 0.2 0.1125 rpy=1.57 0 0
