Commit message: Remove other collision groups since we just use a giant bounding box around the table.

File: data/furniture/uw_demo_table.urdf (robot description, URDF)
Before this commit: robot conference_table, 1 links, 0 joints
Links:
- link base_link: geometry collision box size=1.8288 0.762 0.74295; visual box size=0.06 0.66 0.025

Commit message: Changed table collision geometry to three rectangles to avoid use of a bounding box.

File: data/furniture/uw_demo_table.urdf (robot description, URDF)
Before this commit: robot conference_table, 1 links, 0 joints
Links:
- link base_link: geometry collision box size=0.06 0.62 0.663525; collision box size=0.06 0.62 0.663525
