Commit message: updated workspace

File: data/furniture/workspace_feeding_demo.urdf (robot description, URDF)
Before this commit: robot workspace_feeding_demo, 1 links, 0 joints
Links:
- link workspace: geometry collision box size=0.5 1.6 1.2; collision box size=1 0.71 3

Commit message: feeding demo stuff

File: data/furniture/workspace_feeding_demo.urdf (robot description, URDF)
Before this commit: robot workspace_feeding_demo, 1 links, 0 joints
Links:
- link workspace: geometry collision box size=0.6 1.6 1.2; collision box size=1 0.71 3

Commit message: changed workspace and tom

File: data/furniture/workspace_feeding_demo.urdf (robot description, URDF)
Before this commit: robot workspace_feeding_demo, 1 links, 0 joints
Links:
- link workspace: geometry collision box size=0.6 1.6 1.2; collision box size=2.5 2.5 0.1

File: data/objects/tom.urdf (robot description, URDF)
Before this commit: robot tom, 1 links, 0 joints
Links:
- link base_link: geometry collision box size=1.745 1.3 3; collision mesh filename=tom.dae scale=0.8 0.8 0.8
