Commit message: Fix typo in last commit.

File: data/furniture/sniyaz_bin_table.urdf (robot description, URDF)
Before this commit: robot sniyaz_bin_table, 1 links, 0 joints
Links:
- link base_link: geometry collision box size=0.06 0.62 0.33176; collision box size=0.06 0.62 0.33176

Commit message: Make bin pick table half as deep

File: data/furniture/sniyaz_bin_table.urdf (robot description, URDF)
Before this commit: robot sniyaz_bin_table, 1 links, 0 joints
Links:
- link base_link: geometry collision box size=0.06 0.31 0.33176; collision box size=0.06 0.31 0.33176
