Commit message: updated wheelchair urdf

File: data/furniture/wheelchair.urdf (robot description, URDF)
Before this commit: robot wheelchair, 1 links, 0 joints
Links:
- link base_link: geometry collision mesh filename=wheelchair_collision.stl scale=1 1 1; visual mesh filename=wheelchair.dae scale=1 1 1

Commit message: adapted wheelchair, table, plate, mannequin

File: data/furniture/wheelchair.urdf (robot description, URDF)
Before this commit: robot wheelchair, 1 links, 0 joints
Links:
- link base_link: geometry collision mesh filename=wheelchair_collision.stl scale=1 1 1; visual mesh filename=wheelchair_collision.stl scale=1 1 1

File: data/objects/plate.urdf (robot description, URDF)
Before this commit: robot plate, 1 links, 0 joints
Links:
- link plate: geometry collision mesh filename=plate.stl

Commit message: updated tom and wheelchair

File: data/furniture/wheelchair.urdf (robot description, URDF)
Before this commit: robot wheelchair, 1 links, 0 joints
Links:
- link base_link: geometry collision mesh filename=wheelchair_collision.stl scale=1 1 1; visual mesh filename=wheelchair.dae scale=1 1 1

File: data/objects/tom.urdf (robot description, URDF)
Before this commit: robot tom, 1 links, 0 joints
Links:
- link base_link: geometry collision mesh filename=tom.dae scale=0.8 0.8 0.8; visual mesh filename=tom.dae scale=0.8 0.8 0.8

Commit message: changed workspace and wheelchair

File: data/furniture/wheelchair.urdf (robot description, URDF)
Before this commit: robot wheelchair, 1 links, 0 joints
Links:
- link base_link: geometry collision mesh filename=wheelchair_collision.stl scale=1 1 1; visual mesh filename=wheelchair_collision.stl scale=1 1 1

File: data/furniture/workspace_feeding_demo.urdf (robot description, URDF)
Before this commit: robot workspace_feeding_demo, 1 links, 0 joints
Links:
- link workspace: geometry collision box size=0.6 1.6 1.2; collision box size=2.5 2.5 0.1

Commit message: latest demo status for feeding; needs to be cleaned up

File: data/furniture/wheelchair.urdf (robot description, URDF)
Before this commit: robot wheelchair, 1 links, 0 joints
Links:
- link base_link: geometry collision mesh filename=wheelchair_collision.stl scale=1 1 1; visual mesh filename=wheelchair_collision.stl scale=1 1 1

Commit message: Fixed tom collision

File: data/furniture/wheelchair.urdf (robot description, URDF)
Before this commit: robot wheelchair, 1 links, 0 joints
Links:
- link base_link: geometry collision mesh filename=package://pr_assets/data/furniture/wheelchair.dae scale=1 1 1; collision mesh filename=package://pr_assets/data/furniture/wheelchair_collision.stl scale=1 1 1

File: data/objects/tom.urdf (robot description, URDF)
Before this commit: robot tom, 1 links, 0 joints
Links:
- link base_link: geometry collision box size=0.3 0.4 0.5; collision mesh filename=tom.dae scale=0.8 0.8 0.8

Commit message: Updates from Gen3 integration (#49)
* Fix RGBA calculation for wheelchair

* Added emprise table urdf

* Fixed tom collision

Co-authored-by: Janko Ondras <jo339@cornell.edu>
Co-authored-by: RKJenamani <rajatkj11@gmail.com>
Co-authored-by: Ethan Gordon <ekgordon@cs.washington.edu>

File: data/furniture/wheelchair.urdf (robot description, URDF)
Before this commit: robot wheelchair, 1 links, 0 joints
Links:
- link base_link: geometry collision mesh filename=package://pr_assets/data/furniture/wheelchair.dae scale=1 1 1; collision mesh filename=package://pr_assets/data/furniture/wheelchair_collision.stl scale=1 1 1
